Commit message: Updated mars landscape

File: catkin_ws/src/rover_description/urdf/rover.urdf.xacro (robot description, xacro)
@@ -1,23 +1,7 @@
 <?xml version="1.0" ?>
-<robot name="rover"
-    xmlns:xacro="http://ros.org/wiki/xacro">
-    <link name="base_footprint">
-        <visual>
-            <origin xyz="0 0 0" rpy="0 0 0" />
-            <geometry>
-                <mesh filename="package://rover_description/meshes/rover.stl" scale="0.1 0.1 0.1"/>
-            </geometry>
-        </visual>
-        <collision>
-            <origin xyz="0 0 0.017" rpy="0 0 0" />
-            <geometry>
-                <box size="0.001 0.001 0.001" />
-            </geometry>
-        </collision>
-        <inertial>
-            <origin xyz="0 0 0" />
-            <mass value="0.01" />
-            <inertia ixx="0.001" ixy="0.0" ixz="0.0" iyy="0.001" iyz="0.0" izz="0.001" />
-        </inertial>
-    </link>
+<robot name="rover" xmlns:xacro="http://ros.org/wiki/xacro">
+  <xacro:include filename="$(find rover_description)/urdf/rover_base.urdf.xacro" />
+  <xacro:rover_base wheel_separation="0.235" base_diameter="0.3485">
+    <mesh filename="package://rover_description/meshes/rover.stl" scale="0.1 0.1 0.1"/>
+  </xacro:rover_base>
 </robot>
